Commit message: 初步跑通轮式车模型，但是运动还是有问题

File: akermann/urdf/acuator/front_wheel.urdf.xacro (robot description, xacro)
@@ -12,5 +12,5 @@
                 <geometry>
                     <!--正方体, 单位m-->
-                    <cylinder radius = "${wheel_radius}" length = "0.04"/>
+                    <cylinder radius = "${wheel_radius}" length = "0.14"/>
                 </geometry>
                 <!--材质-->
@@ -26,5 +26,5 @@
                 <geometry>
                     <!--正方体, 单位m-->
-                    <cylinder radius = "${wheel_radius}" length = "0.04"/>
+                    <cylinder radius = "${wheel_radius}" length = "0.14"/>
                 </geometry>
                 <!--材质-->
@@ -35,8 +35,8 @@
             </collision>
             <!--惯性属性-->
-            <xacro:cylinder_inertial m="0.05" r="${wheel_radius}" h="0.04"/>
+            <xacro:cylinder_inertial m="3.0" r="${wheel_radius}" h="0.14"/>
         </link>
         <link name="${front_wheel_name}_steer_link">
-            <xacro:cylinder_inertial m="0.05" r="${wheel_radius}" h="0.04"/>
+            <xacro:cylinder_inertial m="0.01" r="${wheel_radius}" h="0.14"/>
         </link>
         <joint name="${front_wheel_name}_steer_joint" type="revolute">
@@ -48,6 +48,6 @@
             lower="-0.72"
             upper="0.72"
-            effort="0"
-            velocity="0" />
+            effort="5.0"
+            velocity="5.0" />
         </joint>
         <!--机器人关节-->
@@ -63,6 +63,6 @@
         <gazebo reference="${front_wheel_name}_link">
             <material>Gazebo/Yellow</material>
-            <mu1 value="1.2" />
-            <mu2 value="0.9" />
+            <mu1 value="150.0" />
+            <mu2 value="10.0" />
             <kp value="1000000000.0" />
             <kd value="1.0" />

File: akermann/urdf/acuator/rear_wheel.urdf.xacro (robot description, xacro)
@@ -12,5 +12,5 @@
                 <geometry>
                     <!--圆柱体, 单位m-->
-                    <cylinder radius = "${wheel_radius}" length = "0.04"/>
+                    <cylinder radius = "${wheel_radius}" length = "0.14"/>
                 </geometry>
                 <!--材质-->
@@ -26,5 +26,5 @@
                 <geometry>
                     <!--圆柱体, 单位m-->
-                    <cylinder radius = "${wheel_radius}" length = "0.04"/>
+                    <cylinder radius = "${wheel_radius}" length = "0.14"/>
                 </geometry>
                 <!--材质-->
@@ -35,5 +35,5 @@
             </collision>
             <!--惯性属性-->
-            <xacro:cylinder_inertial m="0.05" r="${wheel_radius}" h="0.04"/>
+            <xacro:cylinder_inertial m="3.0" r="${wheel_radius}" h="0.14"/>
         </link>
         <!--机器人关节-->
@@ -45,10 +45,12 @@
             <!--偏移和旋转-->
             <origin xyz="${xyz}" rpy="0.0 0.0 0.0"/>
-             <axis xyz="0.0 1 0.0"/>
+            <dynamics friction="0.8" damping="0.5" />
+            <limit lower="-3.14159" upper="3.14159" effort="200" velocity="-1" />
+            <axis xyz="0.0 1 0.0"/>
         </joint>
         <gazebo reference="${rear_wheel_name}_link">
             <material>Gazebo/Yellow</material>
-            <mu1 value="1.2" />
-            <mu2 value="0.9" />
+            <mu1 value="150.0" />
+            <mu2 value="10.0" />
             <kp value="1000000000.0" />
             <kd value="1.0" />

File: akermann/urdf/base.urdf.xacro (robot description, xacro)
@@ -35,5 +35,5 @@
             </collision>
             <!--惯性属性-->
-            <xacro:box_inertial m="1.0" w="${width}" d="${length}" h="${height}"/>
+            <xacro:box_inertial m="25.0" w="${width}" d="${length}" h="${height}"/>
         </link>
         <link name="base_footprint" />
@@ -69,4 +69,7 @@
             <limit lower="-3" upper="3" effort="200" velocity="20" />
         </joint>
+        <gazebo reference="virtual_steer_link">
+            <material>Gazebo/Yellow</material>
+        </gazebo>
     </xacro:macro>
 </robot>

File: akermann/urdf/plugins/gazebo_control_plugin.xacro (robot description, xacro)
@@ -3,41 +3,60 @@
     <xacro:macro name="gazebo_control_plugin">
         <gazebo>
+            <plugin name="gazebo_ros_joint_state_publisher"
+                filename="libgazebo_ros_joint_state_publisher.so">
+                <update_rate>30.0</update_rate>
+                <joint_name>front_left_wheel_joint</joint_name>
+                <joint_name>front_right_wheel_joint</joint_name>
+                <joint_name>rear_left_wheel_joint</joint_name>
+                <joint_name>rear_right_wheel_joint</joint_name>
+                <joint_name>front_left_wheel_steer_joint</joint_name>
+                <joint_name>front_right_wheel_steer_joint</joint_name>
+                <joint_name>virtual_steering_wheel_joint</joint_name>
+            </plugin>
+        </gazebo>
+        <gazebo>
+            <plugin name="gazebo_ros_joint_pose_trajectory"
+                filename="libgazebo_ros_joint_pose_trajectory.so">
+                <update_rate>2</update_rate>
+            </plugin>
+        </gazebo>
+        <gazebo>
             <plugin name="gazebo_ros_ackermann_drive" filename="libgazebo_ros_ackermann_drive.so">
-            <ros>
-                <namespace>/</namespace>
-                <remapping>cmd_vel:=cmd_vel</remapping>
-                <remapping>odom:=odom</remapping>
-                <remapping>distance:=distance</remapping>
-            </ros>
-            <update_rate>30.0</update_rate>
-            <!-- wheels -->
-            <front_left_joint>front_left_wheel_joint</front_left_joint>
-            <front_right_joint>front_right_wheel_joint</front_right_joint>
-            <rear_left_joint>rear_left_wheel_joint</rear_left_joint>
-            <rear_right_joint>rear_right_wheel_joint</rear_right_joint>
-            <left_steering_joint>front_left_wheel_steer_joint</left_steering_joint>
-            <right_steering_joint>front_right_wheel_steer_joint</right_steering_joint>
-            <steering_wheel_joint>virtual_steering_wheel_joint</steering_wheel_joint>
-            <!-- Max absolute steer angle for tyre in radians-->
-            <!-- Any cmd_vel angular z greater than this would be capped -->
-            <max_steer>0.72</max_steer>
-            <!-- Max absolute steering angle of steering wheel -->
-            <max_steering_angle>7.85</max_steering_angle>
-            <!-- Max absolute linear speed in m/s -->
-            <max_speed>5</max_speed>
-            <!-- PID tuning -->
-            <left_steering_pid_gain>1500 0 1</left_steering_pid_gain>
-            <left_steering_i_range>0 0</left_steering_i_range>
-            <right_steering_pid_gain>1500 0 1</right_steering_pid_gain>
-            <right_steering_i_range>0 0</right_steering_i_range>
-            <linear_velocity_pid_gain>1000 0 1</linear_velocity_pid_gain>
-            <linear_velocity_i_range>0 0</linear_velocity_i_range>
-            <!-- output -->
-            <publish_odom>true</publish_odom>
-            <publish_odom_tf>true</publish_odom_tf>
-            <publish_wheel_tf>false</publish_wheel_tf>
-            <publish_distance>true</publish_distance>
-            <odometry_frame>odom</odometry_frame>
-            <robot_base_frame>base_footprint</robot_base_frame>
+                <ros>
+                    <!-- <namespace>/</namespace> -->
+                    <remapping>cmd_vel:=cmd_vel</remapping>
+                    <remapping>odom:=odom</remapping>
+                    <remapping>distance:=distance</remapping>
+                </ros>
+                <update_rate>30.0</update_rate>
+                <!-- wheels -->
+                <front_left_joint>front_left_wheel_joint</front_left_joint>
+                <front_right_joint>front_right_wheel_joint</front_right_joint>
+                <rear_left_joint>rear_left_wheel_joint</rear_left_joint>
+                <rear_right_joint>rear_right_wheel_joint</rear_right_joint>
+                <left_steering_joint>front_left_wheel_steer_joint</left_steering_joint>
+                <right_steering_joint>front_right_wheel_steer_joint</right_steering_joint>
+                <steering_wheel_joint>virtual_steering_wheel_joint</steering_wheel_joint>
+                <!-- Max absolute steer angle for tyre in radians-->
+                <!-- Any cmd_vel angular z greater than this would be capped -->
+                <max_steer>0.383972</max_steer>
+                <!-- Max absolute steering angle of steering wheel -->
+                <max_steering_angle>1.570796</max_steering_angle>
+                <!-- Max absolute linear speed in m/s -->
+                <max_speed>5</max_speed>
+                <!-- PID tuning -->
+                <left_steering_pid_gain>1500 0 1</left_steering_pid_gain>
+                <left_steering_i_range>0 0</left_steering_i_range>
+                <right_steering_pid_gain>1500 0 1</right_steering_pid_gain>
+                <right_steering_i_range>0 0</right_steering_i_range>
+                <linear_velocity_pid_gain>1000 0 1</linear_velocity_pid_gain>
+                <linear_velocity_i_range>0 0</linear_velocity_i_range>
+                <!-- output -->
+                <publish_odom>true</publish_odom>
+                <publish_odom_tf>true</publish_odom_tf>
+                <publish_wheel_tf>false</publish_wheel_tf>
+                <publish_distance>true</publish_distance>
+                <odometry_frame>odom</odometry_frame>
+                <robot_base_frame>base_footprint</robot_base_frame>
             </plugin>
         </gazebo>

File: akermann/urdf/plugins/gazebo_sensor_plugin.xacro (robot description, xacro)
@@ -20,11 +20,11 @@
                         <horizontal>
                             <samples>360</samples>
-                            <resolution>1</resolution>
-                            <min_angle>0</min_angle>
+                            <resolution>1.0</resolution>
+                            <min_angle>0.0</min_angle>
                             <max_angle>6.28</max_angle>
                         </horizontal>
                     </scan>
                     <range>
-                        <min>1.0</min>
+                        <min>0.1</min>
                         <max>10.0</max>
                         <resolution>0.1</resolution>

File: akermann/urdf/robot.urdf.xacro (robot description, xacro)
@@ -1,7 +1,7 @@
 <?xml version="1.0"?>
 <robot xmlns:xacro="http://www.ros.org/wiki/xacro" name = "robot_name">
-<!-- <xacro:include filename="$(find ackermann)/urdf/sensor/camera.urdf.xacro"/>
-<xacro:include filename="$(find ackermann)/urdf/sensor/imu.urdf.xacro"/>
-<xacro:include filename="$(find ackermann)/urdf/sensor/laser.urdf.xacro"/> -->
+<!-- <xacro:include filename="$(find ackermann)/urdf/sensor/camera.urdf.xacro"/> -->
+<!-- <xacro:include filename="$(find ackermann)/urdf/sensor/imu.urdf.xacro"/> -->
+<xacro:include filename="$(find ackermann)/urdf/sensor/laser.urdf.xacro"/>
 <xacro:include filename="$(find ackermann)/urdf/base.urdf.xacro"/>
 <xacro:include filename="$(find ackermann)/urdf/acuator/front_wheel.urdf.xacro"/>
@@ -9,22 +9,16 @@
 <!-- <xacro:include filename="$(find ackermann)/urdf/acuator/caster.urdf.xacro"/> -->
 <xacro:include filename="$(find ackermann)/urdf/plugins/gazebo_control_plugin.xacro"/>
-<!-- <xacro:include filename="$(find ackermann)/urdf/plugins/gazebo_sensor_plugin.xacro"/> -->
+<xacro:include filename="$(find ackermann)/urdf/plugins/gazebo_sensor_plugin.xacro"/>
 <!-- <xacro:include filename="$(find ackermann)/urdf/ros2_control.xacro"/> -->
-<xacro:base_link length = "0.28" width = "0.184" height = "0.12" wheel_radius = "0.032"/>
-<!-- <xacro:camera_link xyz="0.1 0.0 0.07"/>
-<xacro:imu_link xyz="0.0 0.0 0.02"/>
-<xacro:laser_link xyz="0.0 0.0 0.11"/> -->
-<xacro:rear_wheel_link rear_wheel_name = "rear_left_wheel" wheel_radius = "0.032" xyz="-0.108 0.092 -0.06"/>
-<xacro:rear_wheel_link rear_wheel_name = "rear_right_wheel" wheel_radius = "0.032" xyz="-0.108 -0.092 -0.06"/>
-<xacro:front_wheel_link front_wheel_name = "front_left_wheel" wheel_radius = "0.032" xyz="0.108 0.092 -0.06"/>
-<xacro:front_wheel_link front_wheel_name = "front_right_wheel" wheel_radius = "0.032" xyz="0.108 -0.092 -0.06"/>
+<xacro:base_link length = "0.75" width = "0.3" height = "0.1" wheel_radius = "0.14"/>
+<!-- <xacro:camera_link xyz="0.1 0.0 0.07"/> -->
+<!-- <xacro:imu_link xyz="0.0 0.0 0.02"/> -->
+<xacro:laser_link xyz="0.0 0.0 0.11"/>
+<xacro:rear_wheel_link rear_wheel_name = "rear_left_wheel" wheel_radius = "0.14" xyz="-0.34058 0.24619 -0.1535"/>
+<xacro:rear_wheel_link rear_wheel_name = "rear_right_wheel" wheel_radius = "0.14" xyz="-0.34058 -0.24619 -0.1535"/>
+<xacro:front_wheel_link front_wheel_name = "front_left_wheel" wheel_radius = "0.14" xyz="0.34058 0.24619 -0.1535"/>
+<xacro:front_wheel_link front_wheel_name = "front_right_wheel" wheel_radius = "0.14" xyz="0.34058 -0.24619 -0.1535"/>
 <xacro:gazebo_control_plugin/>
-<gazebo>
-    <plugin name="gazebo_ros_joint_pose_trajectory"
-        filename="libgazebo_ros_joint_pose_trajectory.so">
-        <update_rate>2</update_rate>
-    </plugin>
-</gazebo>
-<!-- <xacro:gazebo_sensor_plugin/>
-<xacro:gazebo_ros2_control_system/> -->
+<xacro:gazebo_sensor_plugin/>
+<!-- <xacro:gazebo_ros2_control_system/> -->
 </robot>

Commit message: 增加建图模块、修改仿真小车结构

File: akermann/urdf/acuator/front_wheel.urdf.xacro (robot description, xacro)
@@ -45,8 +45,9 @@
             <origin rpy="0 0 0" xyz="${xyz}"/>
             <axis xyz="0 0 1"/>
+            <dynamics damping="0.5" />
             <limit
             lower="-0.72"
             upper="0.72"
-            effort="100.0"
+            effort="75.0"
             velocity="5.0" />
         </joint>
@@ -59,5 +60,5 @@
             <!--偏移和旋转-->
             <origin xyz="0.0 0.0 0.0" rpy="0.0 0.0 0.0"/>
-             <axis xyz="0.0 1 0.0"/>
+            <axis xyz="0.0 1 0.0"/>
         </joint>
         <gazebo reference="${front_wheel_name}_link">

File: akermann/urdf/base.urdf.xacro (robot description, xacro)
@@ -67,5 +67,5 @@
             <child link="virtual_steer_link" />
             <axis xyz="-1 0 0" />
-            <limit lower="-3" upper="3" effort="200" velocity="20" />
+            <limit lower="-3.14159" upper="3.14159" effort="200" velocity="20" />
         </joint>
         <gazebo reference="virtual_steer_link">

File: akermann/urdf/plugins/gazebo_control_plugin.xacro (robot description, xacro)
@@ -40,5 +40,5 @@
                 <!-- Max absolute steer angle for tyre in radians-->
                 <!-- Any cmd_vel angular z greater than this would be capped -->
-                <max_steer>0.383972</max_steer>
+                <max_steer>0.72</max_steer>
                 <!-- Max absolute steering angle of steering wheel -->
                 <max_steering_angle>1.570796</max_steering_angle>

File: akermann/urdf/plugins/gazebo_sensor_plugin.xacro (robot description, xacro)
@@ -38,4 +38,72 @@
             </sensor>
         </gazebo>
+        <gazebo reference="imu_link">
+            <sensor name="imu_sensor" type="imu">
+                <plugin filename="libgazebo_ros_imu_sensor.so" name="imu_plugin">
+                    <ros>
+                        <namespace>/</namespace>
+                        <remapping>~/out:=imu</remapping>
+                    </ros>
+                    <initial_orientation_as_reference>false</initial_orientation_as_reference>
+                    </plugin>
+                    <always_on>true</always_on>
+                    <update_rate>50.0</update_rate>
+                    <visualize>true</visualize>
+                    <imu>
+                    <angular_velocity>
+                        <x>
+                        <noise type="gaussian">
+                            <mean>0.0</mean>
+                            <stddev>2e-4</stddev>
+                            <bias_mean>0.0000075</bias_mean>
+                            <bias_stddev>0.0000008</bias_stddev>
+                        </noise>
+                        </x>
+                        <y>
+                        <noise type="gaussian">
+                            <mean>0.0</mean>
+                            <stddev>2e-4</stddev>
+                            <bias_mean>0.0000075</bias_mean>
+                            <bias_stddev>0.0000008</bias_stddev>
+                        </noise>
+                        </y>
+                        <z>
+                        <noise type="gaussian">
+                            <mean>0.0</mean>
+                            <stddev>2e-4</stddev>
+                            <bias_mean>0.0000075</bias_mean>
+                            <bias_stddev>0.0000008</bias_stddev>
+                        </noise>
+                        </z>
+                    </angular_velocity>
+                    <linear_acceleration>
+                        <x>
+                        <noise type="gaussian">
+                            <mean>0.0</mean>
+                            <stddev>1.7e-2</stddev>
+                            <bias_mean>0.1</bias_mean>
+                            <bias_stddev>0.001</bias_stddev>
+                        </noise>
+                        </x>
+                        <y>
+                        <noise type="gaussian">
+                            <mean>0.0</mean>
+                            <stddev>1.7e-2</stddev>
+                            <bias_mean>0.1</bias_mean>
+                            <bias_stddev>0.001</bias_stddev>
+                        </noise>
+                        </y>
+                        <z>
+                        <noise type="gaussian">
+                            <mean>0.0</mean>
+                            <stddev>1.7e-2</stddev>
+                            <bias_mean>0.1</bias_mean>
+                            <bias_stddev>0.001</bias_stddev>
+                        </noise>
+                        </z>
+                    </linear_acceleration>
+                    </imu>
+                </sensor>
+            </gazebo>
     </xacro:macro>
 </robot>

File: akermann/urdf/robot.urdf.xacro (robot description, xacro)
@@ -2,5 +2,5 @@
 <robot xmlns:xacro="http://www.ros.org/wiki/xacro" name = "robot_name">
 <!-- <xacro:include filename="$(find ackermann)/urdf/sensor/camera.urdf.xacro"/> -->
-<!-- <xacro:include filename="$(find ackermann)/urdf/sensor/imu.urdf.xacro"/> -->
+<xacro:include filename="$(find ackermann)/urdf/sensor/imu.urdf.xacro"/>
 <xacro:include filename="$(find ackermann)/urdf/sensor/laser.urdf.xacro"/>
 <xacro:include filename="$(find ackermann)/urdf/base.urdf.xacro"/>
@@ -13,5 +13,5 @@
 <xacro:base_link length = "0.75" width = "0.3" height = "0.1" wheel_radius = "0.14"/>
 <!-- <xacro:camera_link xyz="0.1 0.0 0.07"/> -->
-<!-- <xacro:imu_link xyz="0.0 0.0 0.02"/> -->
+<xacro:imu_link xyz="0.1 0.0 0.051"/>
 <xacro:laser_link xyz="0.0 0.0 0.11"/>
 <xacro:rear_wheel_link rear_wheel_name = "rear_left_wheel" wheel_radius = "0.14" xyz="-0.34058 0.24619 -0.1535"/>

File: akermann/urdf/sensor/imu.urdf.xacro (robot description, xacro)
@@ -45,4 +45,7 @@
             <origin xyz="${xyz}" rpy="0.0 0.0 0.0"/>
         </joint>
+        <gazebo reference="imu_link">
+            <material>Gazebo/Black</material>
+        </gazebo>
     </xacro:macro>
 </robot>
