Commit message: 命名空间隔离、控制器调整为RPP

File: akermann/urdf/acuator/front_wheel.urdf.xacro (robot description, xacro)
@@ -2,7 +2,7 @@
 <robot xmlns:xacro="http://www.ros.org/wiki/xacro">
     <xacro:include filename="$(find ackermann)/urdf/common_inertial.xacro"/>
-    <xacro:macro name="front_wheel_link" params="front_wheel_name wheel_radius xyz">
+    <xacro:macro name="front_wheel_link" params="robot_name front_wheel_name wheel_radius xyz">
         <!--机器人${front_wheel_name}-->
-        <link name="${front_wheel_name}_link">
+        <link name="${robot_name}_${front_wheel_name}_link">
             <!--外观描述-->
             <visual>
@@ -37,10 +37,10 @@
             <xacro:cylinder_inertial m="3.0" r="${wheel_radius}" h="0.14"/>
         </link>
-        <link name="${front_wheel_name}_steer_link">
+        <link name="${robot_name}_${front_wheel_name}_steer_link">
             <xacro:cylinder_inertial m="0.01" r="${wheel_radius}" h="0.14"/>
         </link>
-        <joint name="${front_wheel_name}_steer_joint" type="revolute">
-            <parent link="base_link"/>
-            <child link="${front_wheel_name}_steer_link"/>
+        <joint name="${robot_name}_${front_wheel_name}_steer_joint" type="revolute">
+            <parent link="${robot_name}_base_link"/>
+            <child link="${robot_name}_${front_wheel_name}_steer_link"/>
             <origin rpy="0 0 0" xyz="${xyz}"/>
             <axis xyz="0 0 1"/>
@@ -53,14 +53,14 @@
         </joint>
         <!--机器人关节-->
-        <joint name="${front_wheel_name}_joint" type="continuous">
+        <joint name="${robot_name}_${front_wheel_name}_joint" type="continuous">
             <!--父链接-->
-            <parent link="${front_wheel_name}_steer_link"/>
+            <parent link="${robot_name}_${front_wheel_name}_steer_link"/>
             <!--子链接-->
-            <child link="${front_wheel_name}_link"/>
+            <child link="${robot_name}_${front_wheel_name}_link"/>
             <!--偏移和旋转-->
             <origin xyz="0.0 0.0 0.0" rpy="0.0 0.0 0.0"/>
             <axis xyz="0.0 1 0.0"/>
         </joint>
-        <gazebo reference="${front_wheel_name}_link">
+        <gazebo reference="${robot_name}_${front_wheel_name}_link">
             <material>Gazebo/Yellow</material>
             <mu1 value="150.0" />

File: akermann/urdf/acuator/rear_wheel.urdf.xacro (robot description, xacro)
@@ -2,7 +2,7 @@
 <robot xmlns:xacro="http://www.ros.org/wiki/xacro">
     <xacro:include filename="$(find ackermann)/urdf/common_inertial.xacro"/>
-    <xacro:macro name="rear_wheel_link" params="rear_wheel_name wheel_radius xyz">
+    <xacro:macro name="rear_wheel_link" params="robot_name rear_wheel_name wheel_radius xyz">
         <!--机器人${rear_wheel_name}-->
-        <link name="${rear_wheel_name}_link">
+        <link name="${robot_name}_${rear_wheel_name}_link">
             <!--外观描述-->
             <visual>
@@ -38,9 +38,9 @@
         </link>
         <!--机器人关节-->
-        <joint name="${rear_wheel_name}_joint" type="continuous">
+        <joint name="${robot_name}_${rear_wheel_name}_joint" type="continuous">
             <!--父链接-->
-            <parent link="base_link"/>
+            <parent link="${robot_name}_base_link"/>
             <!--子链接-->
-            <child link="${rear_wheel_name}_link"/>
+            <child link="${robot_name}_${rear_wheel_name}_link"/>
             <!--偏移和旋转-->
             <origin xyz="${xyz}" rpy="0.0 0.0 0.0"/>
@@ -49,5 +49,5 @@
             <axis xyz="0.0 1 0.0"/>
         </joint>
-        <gazebo reference="${rear_wheel_name}_link">
+        <gazebo reference="${robot_name}_${rear_wheel_name}_link">
             <material>Gazebo/Yellow</material>
             <mu1 value="150.0" />

File: akermann/urdf/base.urdf.xacro (robot description, xacro)
@@ -2,7 +2,7 @@
 <robot xmlns:xacro="http://www.ros.org/wiki/xacro" name="robot_name">
     <xacro:include filename="$(find ackermann)/urdf/common_inertial.xacro"/>
-    <xacro:macro name="base_link" params="length width height wheel_radius">
+    <xacro:macro name="base_link" params="robot_name length width height wheel_radius">
         <!--机器人身体部分-->
-        <link name="base_link">
+        <link name="${robot_name}_base_link">
             <!--外观描述-->
             <visual>
@@ -37,14 +37,14 @@
             <xacro:box_inertial m="25.0" w="${width}" d="${length}" h="${height}"/>
         </link>
-        <link name="base_footprint" />
-        <joint name="base_joint" type="fixed">
+        <link name="${robot_name}_base_footprint" />
+        <joint name="${robot_name}_base_joint" type="fixed">
             <!--父链接-->
-            <parent link="base_footprint"/>
+            <parent link="${robot_name}_base_footprint"/>
             <!--子链接-->
-            <child link="base_link"/>
+            <child link="${robot_name}_base_link"/>
             <!--偏移和旋转-->
             <origin xyz="0.0 0.0 ${height / 2.0 + wheel_radius - 0.001}" rpy="0.0 0.0 0.0"/>
         </joint>
-        <link name="virtual_steer_link">
+        <link name="${robot_name}_virtual_steer_link">
             <visual>
                 <origin xyz="0.0 0.0 0.0" rpy="0.0 0.0 0.0" />
@@ -62,12 +62,12 @@
             </inertial>
         </link>
-        <joint name="virtual_steering_wheel_joint" type="revolute">
+        <joint name="${robot_name}_virtual_steering_wheel_joint" type="revolute">
             <origin xyz="0.12 0.0 0.0" rpy="0.0 0.0 0.0" />
-            <parent link="base_link" />
-            <child link="virtual_steer_link" />
+            <parent link="${robot_name}_base_link" />
+            <child link="${robot_name}_virtual_steer_link" />
             <axis xyz="-1 0 0" />
             <limit lower="-3.14159" upper="3.14159" effort="200" velocity="20" />
         </joint>
-        <gazebo reference="virtual_steer_link">
+        <gazebo reference="${robot_name}_virtual_steer_link">
             <material>Gazebo/Yellow</material>
         </gazebo>

File: akermann/urdf/plugins/gazebo_control_plugin.xacro (robot description, xacro)
@@ -1,16 +1,19 @@
 <?xml version = "1.0"?>
 <robot xmlns:xacro="http://www.ros.org/wiki/xacro">
-    <xacro:macro name="gazebo_control_plugin">
+    <xacro:macro name="gazebo_control_plugin" params="robot_name">
         <gazebo>
             <plugin name="gazebo_ros_joint_state_publisher"
                 filename="libgazebo_ros_joint_state_publisher.so">
+                <ros>
+                    <namespace>${robot_name}</namespace>
+                </ros>
                 <update_rate>30.0</update_rate>
-                <joint_name>front_left_wheel_joint</joint_name>
-                <joint_name>front_right_wheel_joint</joint_name>
-                <joint_name>rear_left_wheel_joint</joint_name>
-                <joint_name>rear_right_wheel_joint</joint_name>
-                <joint_name>front_left_wheel_steer_joint</joint_name>
-                <joint_name>front_right_wheel_steer_joint</joint_name>
-                <joint_name>virtual_steering_wheel_joint</joint_name>
+                <joint_name>${robot_name}_front_left_wheel_joint</joint_name>
+                <joint_name>${robot_name}_front_right_wheel_joint</joint_name>
+                <joint_name>${robot_name}_rear_left_wheel_joint</joint_name>
+                <joint_name>${robot_name}_rear_right_wheel_joint</joint_name>
+                <joint_name>${robot_name}_front_left_wheel_steer_joint</joint_name>
+                <joint_name>${robot_name}_front_right_wheel_steer_joint</joint_name>
+                <joint_name>${robot_name}_virtual_steering_wheel_joint</joint_name>
             </plugin>
         </gazebo>
@@ -18,4 +21,7 @@
             <plugin name="gazebo_ros_joint_pose_trajectory"
                 filename="libgazebo_ros_joint_pose_trajectory.so">
+                <ros>
+                    <namespace>${robot_name}</namespace>
+                </ros>
                 <update_rate>2</update_rate>
             </plugin>
@@ -24,5 +30,5 @@
             <plugin name="gazebo_ros_ackermann_drive" filename="libgazebo_ros_ackermann_drive.so">
                 <ros>
-                    <!-- <namespace>/</namespace> -->
+                    <namespace>${robot_name}</namespace>
                     <remapping>cmd_vel:=cmd_vel</remapping>
                     <remapping>odom:=odom</remapping>
@@ -31,11 +37,11 @@
                 <update_rate>30.0</update_rate>
                 <!-- wheels -->
-                <front_left_joint>front_left_wheel_joint</front_left_joint>
-                <front_right_joint>front_right_wheel_joint</front_right_joint>
-                <rear_left_joint>rear_left_wheel_joint</rear_left_joint>
-                <rear_right_joint>rear_right_wheel_joint</rear_right_joint>
-                <left_steering_joint>front_left_wheel_steer_joint</left_steering_joint>
-                <right_steering_joint>front_right_wheel_steer_joint</right_steering_joint>
-                <steering_wheel_joint>virtual_steering_wheel_joint</steering_wheel_joint>
+                <front_left_joint>${robot_name}_front_left_wheel_joint</front_left_joint>
+                <front_right_joint>${robot_name}_front_right_wheel_joint</front_right_joint>
+                <rear_left_joint>${robot_name}_rear_left_wheel_joint</rear_left_joint>
+                <rear_right_joint>${robot_name}_rear_right_wheel_joint</rear_right_joint>
+                <left_steering_joint>${robot_name}_front_left_wheel_steer_joint</left_steering_joint>
+                <right_steering_joint>${robot_name}_front_right_wheel_steer_joint</right_steering_joint>
+                <steering_wheel_joint>${robot_name}_virtual_steering_wheel_joint</steering_wheel_joint>
                 <!-- Max absolute steer angle for tyre in radians-->
                 <!-- Any cmd_vel angular z greater than this would be capped -->
@@ -57,6 +63,6 @@
                 <publish_wheel_tf>false</publish_wheel_tf>
                 <publish_distance>true</publish_distance>
-                <odometry_frame>odom</odometry_frame>
-                <robot_base_frame>base_footprint</robot_base_frame>
+                <odometry_frame>${robot_name}_odom</odometry_frame>
+                <robot_base_frame>${robot_name}_base_footprint</robot_base_frame>
             </plugin>
         </gazebo>

File: akermann/urdf/plugins/gazebo_sensor_plugin.xacro (robot description, xacro)
@@ -1,14 +1,14 @@
 <?xml version = "1.0"?>
 <robot xmlns:xacro="http://www.ros.org/wiki/xacro">
-    <xacro:macro name="gazebo_sensor_plugin">
-        <gazebo reference = "laser_link">
+    <xacro:macro name="gazebo_sensor_plugin" params="robot_name">
+        <gazebo reference = "${robot_name}_laser_link">
             <sensor name = "laserscan" type = "ray">
                 <plugin name = "laserscan" filename = "libgazebo_ros_ray_sensor.so">
                     <ros>
-                        <namespace>/</namespace>
+                        <namespace>${robot_name}</namespace>
                         <remapping>~/out:=scan</remapping>
                     </ros>
                     <output_type>sensor_msgs/LaserScan</output_type>
-                    <frameName>laser_link</frameName>
+                    <frameName>${robot_name}_laser_link</frameName>
                 </plugin>
                 <always_on>true</always_on>
@@ -38,9 +38,9 @@
             </sensor>
         </gazebo>
-        <gazebo reference="imu_link">
+        <gazebo reference="${robot_name}_imu_link">
             <sensor name="imu_sensor" type="imu">
                 <plugin filename="libgazebo_ros_imu_sensor.so" name="imu_plugin">
                     <ros>
-                        <namespace>/</namespace>
+                        <namespace>${robot_name}</namespace>
                         <remapping>~/out:=imu</remapping>
                     </ros>

File: akermann/urdf/robot.urdf.xacro (robot description, xacro)
@@ -1,4 +1,5 @@
 <?xml version="1.0"?>
-<robot xmlns:xacro="http://www.ros.org/wiki/xacro" name = "robot_name">
+<robot xmlns:xacro="http://www.ros.org/wiki/xacro" name = "robot">
+<xacro:arg name="robot_name" default="robot1"/>
 <!-- <xacro:include filename="$(find ackermann)/urdf/sensor/camera.urdf.xacro"/> -->
 <xacro:include filename="$(find ackermann)/urdf/sensor/imu.urdf.xacro"/>
@@ -11,14 +12,14 @@
 <xacro:include filename="$(find ackermann)/urdf/plugins/gazebo_sensor_plugin.xacro"/>
 <!-- <xacro:include filename="$(find ackermann)/urdf/ros2_control.xacro"/> -->
-<xacro:base_link length = "0.75" width = "0.3" height = "0.1" wheel_radius = "0.14"/>
+<xacro:base_link robot_name = "$(arg robot_name)" length = "0.75" width = "0.3" height = "0.1" wheel_radius = "0.14"/>
 <!-- <xacro:camera_link xyz="0.1 0.0 0.07"/> -->
-<xacro:imu_link xyz="0.1 0.0 0.051"/>
-<xacro:laser_link xyz="0.0 0.0 0.11"/>
-<xacro:rear_wheel_link rear_wheel_name = "rear_left_wheel" wheel_radius = "0.14" xyz="-0.34058 0.24619 -0.1535"/>
-<xacro:rear_wheel_link rear_wheel_name = "rear_right_wheel" wheel_radius = "0.14" xyz="-0.34058 -0.24619 -0.1535"/>
-<xacro:front_wheel_link front_wheel_name = "front_left_wheel" wheel_radius = "0.14" xyz="0.34058 0.24619 -0.1535"/>
-<xacro:front_wheel_link front_wheel_name = "front_right_wheel" wheel_radius = "0.14" xyz="0.34058 -0.24619 -0.1535"/>
-<xacro:gazebo_control_plugin/>
-<xacro:gazebo_sensor_plugin/>
+<xacro:imu_link robot_name = "$(arg robot_name)" xyz="0.1 0.0 0.051"/>
+<xacro:laser_link robot_name = "$(arg robot_name)" xyz="0.0 0.0 0.11"/>
+<xacro:rear_wheel_link robot_name = "$(arg robot_name)" rear_wheel_name = "rear_left_wheel" wheel_radius = "0.14" xyz="-0.34058 0.24619 -0.1535"/>
+<xacro:rear_wheel_link robot_name = "$(arg robot_name)" rear_wheel_name = "rear_right_wheel" wheel_radius = "0.14" xyz="-0.34058 -0.24619 -0.1535"/>
+<xacro:front_wheel_link robot_name = "$(arg robot_name)" front_wheel_name = "front_left_wheel" wheel_radius = "0.14" xyz="0.34058 0.24619 -0.1535"/>
+<xacro:front_wheel_link robot_name = "$(arg robot_name)" front_wheel_name = "front_right_wheel" wheel_radius = "0.14" xyz="0.34058 -0.24619 -0.1535"/>
+<xacro:gazebo_control_plugin robot_name = "$(arg robot_name)"/>
+<xacro:gazebo_sensor_plugin robot_name = "$(arg robot_name)"/>
 <!-- <xacro:gazebo_ros2_control_system/> -->
 </robot>

File: akermann/urdf/sensor/imu.urdf.xacro (robot description, xacro)
@@ -1,7 +1,7 @@
 <?xml version="1.0"?>
 <robot xmlns:xacro="http://www.ros.org/wiki/xacro">
-    <xacro:macro name="imu_link" params="xyz">
+    <xacro:macro name="imu_link" params="robot_name xyz">
         <!--机器人IMU-->
-        <link name="imu_link">
+        <link name="${robot_name}_imu_link">
             <!--外观描述-->
             <visual>
@@ -37,13 +37,13 @@
         </link>
         <!--机器人关节-->
-        <joint name="imu_joint" type="fixed">
+        <joint name="${robot_name}_imu_joint" type="fixed">
             <!--父链接-->
-            <parent link="base_link"/>
+            <parent link="${robot_name}_base_link"/>
             <!--子链接-->
-            <child link="imu_link"/>
+            <child link="${robot_name}_imu_link"/>
             <!--偏移和旋转-->
             <origin xyz="${xyz}" rpy="0.0 0.0 0.0"/>
         </joint>
-        <gazebo reference="imu_link">
+        <gazebo reference="${robot_name}_imu_link">
             <material>Gazebo/Black</material>
         </gazebo>

File: akermann/urdf/sensor/laser.urdf.xacro (robot description, xacro)
@@ -1,7 +1,7 @@
 <?xml version="1.0"?>
 <robot xmlns:xacro="http://www.ros.org/wiki/xacro">
-    <xacro:macro name="laser_link" params="xyz">
+    <xacro:macro name="laser_link" params="robot_name xyz">
         <!--机器人laser-->
-        <link name="laser_cylinder_link">
+        <link name="${robot_name}_laser_cylinder_link">
             <!--外观描述-->
             <visual>
@@ -36,5 +36,5 @@
             <xacro:cylinder_inertial m="0.05" r="0.01" h="0.2"/>
         </link>
-        <link name="laser_link">
+        <link name="${robot_name}_laser_link">
             <!--外观描述-->
             <visual>
@@ -70,22 +70,22 @@
         </link>
         <!--机器人关节-->
-        <joint name="laser_joint" type="fixed">
+        <joint name="${robot_name}_laser_joint" type="fixed">
             <!--父链接-->
-            <parent link="laser_cylinder_link"/>
+            <parent link="${robot_name}_laser_cylinder_link"/>
             <!--子链接-->
-            <child link="laser_link"/>
+            <child link="${robot_name}_laser_link"/>
             <!--偏移和旋转-->
             <origin xyz="0 0 0.1" rpy="0.0 0.0 0.0"/>
         </joint>
         <!--机器人关节-->
-        <joint name="laser_cylinder_joint" type="fixed">
+        <joint name="${robot_name}_laser_cylinder_joint" type="fixed">
             <!--父链接-->
-            <parent link="base_link"/>
+            <parent link="${robot_name}_base_link"/>
             <!--子链接-->
-            <child link="laser_cylinder_link"/>
+            <child link="${robot_name}_laser_cylinder_link"/>
             <!--偏移和旋转-->
             <origin xyz="${xyz}" rpy="0.0 0.0 0.0"/>
         </joint>
-        <gazebo reference="laser_cylinder_link">
+        <gazebo reference="${robot_name}_laser_cylinder_link">
             <material>Gazebo/Black</material>
         </gazebo>
